Commit message: Removed world framed and changed standard localization to amcl

File: mobrob_robin_description/robots/test.urdf (robot description, URDF)
Before this commit: robot mobrob_robin, 14 links, 13 joints
Links:
- removed link world
Joints:
- removed joint odom_joint

File: mobrob_robin_description/urdf/mobrob_robin_base/base.urdf.xacro (robot description, xacro)
@@ -3,12 +3,4 @@
    <xacro:include filename="$(find mobrob_robin_description)/urdf/mobrob_robin_base/base.transmission.xacro" />
    <xacro:macro name="base" params="">
-      <link name="world" />
-      <joint name="odom_joint" type="fixed">
-         <xacro:if value="${simulated}">
-            <origin xyz="$(arg ofx) $(arg ofy) $(arg ofz)" rpy="0 0 0" />
-         </xacro:if>
-         <parent link="world" />
-         <child link="odom" />
-      </joint>
       <link name="odom">
          <inertial>
