Commit message: Updated installation instructions. Removed dwa_spline_local_planner because it is not robot specific and will be added to ros_common_robin later. Added packages for gazebo simulation of the mobrob_robin robot.

File: mobrob_robin_description/urdf/mobrob_robin_base/base.urdf.xacro (robot description, xacro)
@@ -57,42 +57,298 @@
          <child link="base_link" />
       </joint>
-      <link name="base_link">
-         <inertial>
-            <mass value="1.0" />
-            <origin xyz="0.0 0.0 0.0" rpy="0 0 0" />
-            <inertia ixx="0.1" ixy="0.0" ixz="0.0" iyy="0.1" iyz="0.0" izz="0.1" />
-         </inertial>
-         <!-- z verschiebung = Abstand von Boden zu Motor achse + Rad Radius -->
-         <visual>
-            <origin xyz="0 0 0" rpy="1.57079 0 1.57079" />
-            <geometry>
-               <mesh filename="package://mobrob_robin_description/meshes/mobrob.dae" scale="0.001 0.001 0.001" />
-            </geometry>
-            <material name="test">
-               <color rgba="0.5 0.5 0.5 1.0" />
-            </material>
-         </visual>
-         <collision>
-            <origin xyz="0.0 0.0 0.36" rpy="0 0 0" />
-            <geometry>
-               <cylinder length="0.71" radius="0.425" />
-            </geometry>
-         </collision>
-      </link>
-      <joint name="base_mass_joint" type="fixed">
-         <origin xyz="0 0 0.4" rpy="0 0 0" />
-         <parent link="base_link" />
-         <child link="base_mass_link" />
-      </joint>
-      <link name="base_mass_link">
-         <inertial>
-            <mass value="80.0" />
-            <origin xyz="0.0 0.0 0.0" rpy="0 0 0" />
-            <inertia ixx="0.5" ixy="0.0" ixz="0.0" iyy="0.5" iyz="0.0" izz="0.5" />
-         </inertial>
-      </link>
-      <xacro:if value="${simulated}">
-         <xacro:omnirob_transmission />
-      </xacro:if>
+  <link name="base_link">
+    <inertial>
+      <mass value="${base_mass}" />
+      <origin xyz="0 0 ${base_height}" />
+      <inertia ixx="${base_ixx}" ixy="0.0" ixz="0.0"
+        iyy="${base_iyy}" iyz="0.0" izz="${base_izz}" />
+    </inertial>
+    <visual>
+      <origin xyz=" 0 0 ${base_1_size_z/2 + base_height}" rpy="0 0 0" />
+      <geometry>
+        <!--<mesh scale="1.0 1.0 1.0 " filename="package://mobrob_robin_description/meshes/mobrob.stl"/>-->
+        <box size="${base_1_size_x} ${base_1_size_y} ${base_1_size_z}" />
+      </geometry>
+      <material name="Gray_light" />
+    </visual>
+    <collision>
+      <origin xyz="0 0 ${base_1_size_z/2}" rpy="0 0 0" />
+      <geometry>
+        <box size="${base_1_size_x} ${base_1_size_y} ${base_1_size_z}" />
+      </geometry>
+    </collision>
+  </link>
+  <joint name="base_upper_joint" type="fixed">
+    <origin xyz="${base_2_size_x / 2 - base_1_size_x / 2} 0 ${base_1_size_z + base_height}" rpy="0 0 0" />
+    <parent link="base_link"/>
+    <child link="base_upper_body" />
+  </joint>
+  <link name="base_upper_body">
+    <inertial>
+      <mass value="0.0001" />
+      <origin xyz="0 0 0.0" />
+      <inertia ixx="0.0001" ixy="0.0" ixz="0.0"
+        iyy="0.0001" iyz="0.0" izz="0.0001" />
+    </inertial>
+    <visual>
+      <origin xyz=" 0 0 ${base_2_size_z/2}" rpy="0 0 0" />
+      <geometry>
+        <box size="${base_2_size_x} ${base_2_size_y} ${base_2_size_z}" />
+        <!--<box size="0.001 0.001 0.001" />-->
+      </geometry>
+      <material name="Gray_light" />
+    </visual>
+    <collision>
+      <origin xyz="0 0 ${base_2_size_z/2}" rpy="0 0 0" />
+      <geometry>
+        <box size="${base_2_size_x} ${base_2_size_y} ${base_2_size_z}" />
+      </geometry>
+    </collision>
+  </link>
+  <!--                         Wheel definition rotation z-axis                                        -->
+  <!--wheel right front rotation z-axis-->
+  <link name="wheel_rf_rot_z">
+    <inertial>
+      <origin xyz="0 0 0"/>
+      <mass value="1.0" />
+      <inertia ixx="0.001" ixy="0.0" ixz="0.0"
+        iyy="0.001" iyz="0.0" izz="0.001" />
+    </inertial>
+    <visual>
+      <origin xyz="0 0 0" rpy="0 0 ${M_PI}" />
+      <geometry>
+        <mesh scale="0.01 0.01 0.01 " filename="package://mobrob_robin_description/meshes/wheel_suspension_small_long.stl"/>
+        <!--<box size="0.01 0.01 0.01" />-->
+      </geometry>
+      <material name="Gray_middle" />
+    </visual>
+    <collision>
+      <origin xyz="0 0 0" rpy="0 0 ${M_PI}" />
+      <geometry>
+        <mesh scale="0.01 0.01 0.01 " filename="package://mobrob_robin_description/meshes/wheel_suspension_small_long.stl"/>
+        <!--<box size="0.01 0.01 0.01" />-->
+      </geometry>
+    </collision>
+  </link>
+    <joint name="wheel_rf_rot_z_joint" type="continuous">
+    <dynamics damping="1.0" friction="0.0" />
+    <origin xyz="${wheel_rf_offset_x} ${wheel_rf_offset_y}  ${base_height}" rpy="0 0 0"/>
+    <parent link="base_link"/>
+    <child link="wheel_rf_rot_z"/>
+    <axis xyz="0 0 1"/>
+  </joint>
+    <!--wheel left back rotation z-axis-->
+  <link name="wheel_lb_rot_z">
+    <inertial>
+      <origin xyz="0 0 0"/>
+      <mass value="1.0" />
+      <inertia ixx="0.001" ixy="0.0" ixz="0.0"
+        iyy="0.001" iyz="0.0" izz="0.001" />
+    </inertial>
+    <visual>
+      <origin xyz="0 0 0" rpy="0 0 0" />
+      <geometry>
+        <mesh scale="0.01 0.01 0.01 " filename="package://mobrob_robin_description/meshes/wheel_suspension_small_long.stl"/>
+        <!--<box size="0.01 0.01 0.01" />-->
+      </geometry>
+      <material name="Gray_middle" />
+    </visual>
+    <collision>
+      <origin xyz="0 0 0" rpy="0 0 0" />
+      <geometry>
+        <mesh scale="0.01 0.01 0.01 " filename="package://mobrob_robin_description/meshes/wheel_suspension_small_long.stl"/>
+        <!--<box size="0.01 0.01 0.01" />-->
+      </geometry>
+    </collision>
+  </link>
+   <joint name="wheel_lb_rot_z_joint" type="continuous">
+   <dynamics damping="1.0" friction="0.0" />
+    <origin xyz="${wheel_lb_offset_x} ${wheel_lb_offset_y} ${base_height}" rpy="0 0 0"/>
+    <parent link="base_link"/>
+    <child link="wheel_lb_rot_z"/>
+    <axis xyz="0 0 1"/>
+  </joint>
+  <!--wheel left front rotation z-axis-->
+  <link name="wheel_lf_rot_z">
+    <inertial>
+      <origin xyz="0 0 0"/>
+      <mass value="1.0" />
+      <inertia ixx="0.001" ixy="0.0" ixz="0.0"
+        iyy="0.001" iyz="0.0" izz="0.001" />
+    </inertial>
+    <visual>
+      <origin xyz="0 0 0" rpy="0 0 0" />
+      <geometry>
+        <mesh scale="0.01 0.01 0.01 " filename="package://mobrob_robin_description/meshes/wheel_suspension_big.stl"/>
+        <!--<box size="0.01 0.01 0.01" />-->
+      </geometry>
+      <material name="Gray_middle" />
+    </visual>
+    <collision>
+      <origin xyz="0 0 0" rpy="0 0 0" />
+      <geometry>
+        <mesh scale="0.01 0.01 0.01 " filename="package://mobrob_robin_description/meshes/wheel_suspension_big.stl"/>
+        <!--<box size="0.01 0.01 0.01" />-->
+      </geometry>
+    </collision>
+  </link>
+  <joint name="wheel_lf_rot_z_joint" type="continuous">
+  <dynamics damping="1.0" friction="0.0" />
+    <origin xyz="${wheel_lf_offset_x} ${wheel_lf_offset_y} ${base_height}" rpy="0 0 0"/>
+    <parent link="base_link"/>
+    <child link="wheel_lf_rot_z"/>
+    <axis xyz="0 0 1"/>
+  </joint>
+  <!--wheel right back rotation z-axis-->
+  <link name="wheel_rb_rot_z">
+    <inertial>
+      <origin xyz="0 0 0"/>
+      <mass value="0.001" />
+      <inertia ixx="0.001" ixy="0.0" ixz="0.0"
+        iyy="0.001" iyz="0.0" izz="0.001" />
+    </inertial>
+    <visual>
+      <origin xyz="0 0 0" rpy="0 0 ${M_PI}" />
+      <geometry>
+        <mesh scale="0.01 0.01 0.01 " filename="package://mobrob_robin_description/meshes/wheel_suspension_big.stl"/>
+        <!--<box size="0.01 0.01 0.01" />-->
+      </geometry>
+      <material name="Gray_middle" />
+    </visual>
+    <collision>
+      <origin xyz="0 0 0" rpy="0 0 ${M_PI}" />
+      <geometry>
+        <mesh scale="0.01 0.01 0.01 " filename="package://mobrob_robin_description/meshes/wheel_suspension_big.stl"/>
+        <!--<box size="0.01 0.01 0.01" />-->
+      </geometry>
+    </collision>
+  </link>
+  <joint name="wheel_rb_rot_z_joint" type="continuous">
+  <dynamics damping="1.0" friction="0.0" />
+    <origin xyz="${wheel_rb_offset_x} ${wheel_rb_offset_y} ${base_height}" rpy="0 0 0"/>
+    <parent link="base_link"/>
+    <child link="wheel_rb_rot_z"/>
+    <axis xyz="0 0 1"/>
+  </joint>
+    <!--                         Wheel definition rotation y-axis                                        -->
+    <!--wheel right front rotation y-axis-->
+    <link name="wheel_rf_rot_y">
+    <inertial>
+      <origin xyz="0 0 0"/>
+      <mass value="${wheel_small_mass}" />
+      <inertia ixx="${wheel_small_ixx}" ixy="0.0" ixz="0.0"
+        iyy="${wheel_small_iyy}" iyz="0.0" izz="${wheel_small_izz}" />
+    </inertial>
+    <visual>
+      <origin xyz="0 0 0" rpy="0 0 ${M_PI/2}" />
+      <geometry>
+        <mesh scale="0.01 0.01 0.01 " filename="package://mobrob_robin_description/meshes/wheel_small.stl"/>
+      </geometry>
+      <material name="Gray_dark" />
+    </visual>
+    <collision>
+      <origin xyz="0 0 0" rpy="${M_PI/2} 0 0" />
+      <geometry>
+        <cylinder radius="${wheel_small_radius}" length = "${wheel_small_length}"/>
+      </geometry>
+    </collision>
+  </link>
+   <joint name="wheel_rf_rot_y_joint" type="continuous">
+   <dynamics damping="1.0" friction="0.0" />
+    <origin xyz="0 0 ${wheel_rf_offset_z}" rpy="0 0 0"/>
+    <parent link="wheel_rf_rot_z"/>
+    <child link="wheel_rf_rot_y"/>
+    <axis xyz="0 1 0"/>
+  </joint>
+     <!--wheel left back rotation y-axis-->
+    <link name="wheel_lb_rot_y">
+    <inertial>
+      <origin xyz="0 0 0"/>
+      <mass value="${wheel_small_mass}" />
+      <inertia ixx="${wheel_small_ixx}" ixy="0.0" ixz="0.0"
+        iyy="${wheel_small_iyy}" iyz="0.0" izz="${wheel_small_izz}" />
+    </inertial>
+    <visual>
+      <origin xyz="0 0 0" rpy="0 0 ${M_PI/2}" />
+      <geometry>
+        <mesh scale="0.01 0.01 0.01 " filename="package://mobrob_robin_description/meshes/wheel_small.stl"/>
+      </geometry>
+      <material name="Gray_dark" />
+    </visual>
+    <collision>
+      <origin xyz="0 0 0" rpy="${M_PI/2} 0 0" />
+      <geometry>
+        <cylinder radius="${wheel_small_radius}" length = "${wheel_small_length}"/>
+      </geometry>
+    </collision>
+  </link>
+   <joint name="wheel_lb_rot_y_joint" type="continuous">
+   <dynamics damping="1.0" friction="0.0" />
+    <origin xyz="0 0 ${wheel_lb_offset_z}" rpy="0 0 0"/>
+    <parent link="wheel_lb_rot_z"/>
+    <child link="wheel_lb_rot_y"/>
+    <axis xyz="0 1 0"/>
+  </joint>
+       <!--wheel left front rotation y-axis-->
+  <link name="wheel_lf_rot_y">
+    <inertial>
+      <origin xyz="0 0 0"/>
+      <mass value="${wheel_big_mass}" />
+      <inertia ixx="${wheel_big_ixx}" ixy="0.0" ixz="0.0"
+        iyy="${wheel_big_iyy}" iyz="0.0" izz="${wheel_big_izz}" />
+    </inertial>
+    <visual>
+      <origin xyz="0 0 0" rpy="0 0 ${M_PI/2}" />
+      <geometry>
+        <mesh scale="0.01 0.01 0.01 " filename="package://mobrob_robin_description/meshes/wheel_big.stl"/>
+      </geometry>
+      <material name="Gray_dark" />
+    </visual>
+    <collision>
+      <origin xyz="0 0 0" rpy="${M_PI/2} 0 0" />
+      <geometry>
+        <cylinder radius="${wheel_big_radius}" length = "${wheel_big_length}"/>
+      </geometry>
+    </collision>
+  </link>
+   <joint name="wheel_lf_rot_y_joint" type="continuous">
+   <dynamics damping="1.0" friction="0.0" />
+    <origin xyz="0 0 ${wheel_lf_offset_z}" rpy="0 0 0"/>
+    <parent link="wheel_lf_rot_z"/>
+    <child link="wheel_lf_rot_y"/>
+    <axis xyz="0 1 0"/>
+  </joint>
+         <!--wheel right back rotation y-axis-->
+  <link name="wheel_rb_rot_y">
+    <inertial>
+      <origin xyz="0 0 0"/>
+      <mass value="${wheel_big_mass}" />
+      <inertia ixx="${wheel_big_ixx}" ixy="0.0" ixz="0.0"
+        iyy="${wheel_big_iyy}" iyz="0.0" izz="${wheel_big_izz}" />
+    </inertial>
+    <visual>
+      <origin xyz="0 0 0" rpy="0 0 ${M_PI/2}" />
+      <geometry>
+        <mesh scale="0.01 0.01 0.01 " filename="package://mobrob_robin_description/meshes/wheel_big.stl"/>
+      </geometry>
+      <material name="Gray_dark" />
+    </visual>
+    <collision>
+      <origin xyz="0 0 0" rpy="${M_PI/2} 0 0" />
+      <geometry>
+        <cylinder radius="${wheel_big_radius}" length = "${wheel_big_length}"/>
+      </geometry>
+    </collision>
+  </link>
+   <joint name="wheel_rb_rot_y_joint" type="continuous">
+   <dynamics damping="1.0" friction="0.0" />
+    <origin xyz="0 0 ${wheel_rb_offset_z}" rpy="0 0 0"/>
+    <parent link="wheel_rb_rot_z"/>
+    <child link="wheel_rb_rot_y"/>
+    <axis xyz="0 1 0"/>
+  </joint>
+  <xacro:if value="${simulated}">
+	<xacro:mobrob_transmission />
+  </xacro:if>
    </xacro:macro>
 </robot>

Commit message: Added ultrasound sensors to mobrob description

File: mobrob_robin_description/robots/mobrob.urdf.xacro (robot description, xacro)
@@ -5,3 +5,27 @@
   <xacro:base />
   <xacro:sensor_pls200 />
+  <xacro:ultrasound_sensor parent="base_link" number="0">
+    <insert_block name="ultrasound_sensor0" />
+  </xacro:ultrasound_sensor>
+  <xacro:ultrasound_sensor parent="base_link" number="1">
+    <insert_block name="ultrasound_sensor1" />
+  </xacro:ultrasound_sensor>
+  <xacro:ultrasound_sensor parent="base_link" number="2">
+    <insert_block name="ultrasound_sensor2" />
+  </xacro:ultrasound_sensor>
+  <xacro:ultrasound_sensor parent="base_link" number="3">
+    <insert_block name="ultrasound_sensor3" />
+  </xacro:ultrasound_sensor>
+  <xacro:ultrasound_sensor parent="base_link" number="4">
+    <insert_block name="ultrasound_sensor4" />
+  </xacro:ultrasound_sensor>
+  <xacro:ultrasound_sensor parent="base_link" number="5">
+    <insert_block name="ultrasound_sensor5" />
+  </xacro:ultrasound_sensor>
+  <xacro:ultrasound_sensor parent="base_link" number="6">
+    <insert_block name="ultrasound_sensor6" />
+  </xacro:ultrasound_sensor>
+  <xacro:ultrasound_sensor parent="base_link" number="7">
+    <insert_block name="ultrasound_sensor7" />
+  </xacro:ultrasound_sensor>
 </robot>

File: mobrob_robin_description/urdf/mobrob_robin.library.xacro (robot description, xacro)
@@ -16,3 +16,5 @@
   <!-- Laserscanner -->
   <xacro:include filename="$(find mobrob_robin_description)/urdf/sensors/pls200.urdf.xacro"/>
+  <!-- Ultrasound -->
+  <xacro:include filename="$(find mobrob_robin_description)/urdf/sensors/ultrasound.urdf.xacro"/>
 </robot>

File: mobrob_robin_description/urdf/mobrob_robin.properties.xacro (robot description, xacro)
@@ -103,4 +103,35 @@
   <property name="base_arduino_platform_size_y" value="0.08" />
   <property name="base_arduino_platform_size_z" value="0.003" />
-  <property name="base_arduino_pitch" value="25" /><!--degree-->
+  <property name="base_arduino_pitch" value="25" /><!--degree-->,
+  <property name="ultrasound_z" value="${0.810-0.075}"/>
+  <property name="ultrasound_back_front_y" value="${0.25-0.057}"/> <!--offset for the sensors on the side -->
+  <property name="ultrasound_back_x" value="${-0.3+0.01}" />
+  <property name="ultrasound_front_x" value="${-0.3+0.345-0.01}" />
+  <property name="ultrasound_left_right_y" value="${0.25-0.01}" />
+  <property name="ultrasound_back_side_x" value="${-0.3+0.057}" />
+  <property name="ultrasound_front_side_x" value="${-0.3+0.345-0.057}" />
+  <xacro:property name="ultrasound_sensor0"> <!-- lb back -->
+    <origin xyz="${ultrasound_back_x} ${ultrasound_back_front_y} ${ultrasound_z}" rpy="0 0 ${M_PI}"/>
+  </xacro:property>
+  <xacro:property name="ultrasound_sensor1"> <!-- lb left -->
+    <origin xyz="${ultrasound_back_side_x} ${ultrasound_left_right_y} ${ultrasound_z}" rpy="0 0 ${M_PI/2}"/>
+  </xacro:property>
+  <xacro:property name="ultrasound_sensor2"> <!-- lf left -->
+    <origin xyz="${ultrasound_front_side_x} ${ultrasound_left_right_y} ${ultrasound_z}" rpy="0 0 ${M_PI/2}"/>
+  </xacro:property>
+  <xacro:property name="ultrasound_sensor3"> <!-- lf front -->
+    <origin xyz="${ultrasound_front_x} ${ultrasound_back_front_y} ${ultrasound_z}" rpy="0 0 ${0}"/>
+  </xacro:property>
+  <xacro:property name="ultrasound_sensor4"> <!-- rf front -->
+    <origin xyz="${ultrasound_front_x} ${-ultrasound_back_front_y} ${ultrasound_z}" rpy="0 0 ${0}"/>
+  </xacro:property>
+  <xacro:property name="ultrasound_sensor5"> <!-- rf right -->
+    <origin xyz="${ultrasound_front_side_x} ${-ultrasound_left_right_y} ${ultrasound_z}" rpy="0 0 ${3*M_PI/2}"/>
+  </xacro:property>
+  <xacro:property name="ultrasound_sensor6"> <!-- rb right -->
+    <origin xyz="${ultrasound_back_side_x} ${-ultrasound_left_right_y} ${ultrasound_z}" rpy="0 0 ${3*M_PI/2}"/>
+  </xacro:property>
+  <xacro:property name="ultrasound_sensor7"> <!-- rb back -->
+    <origin xyz="${ultrasound_back_x} ${-ultrasound_back_front_y} ${ultrasound_z}" rpy="0 0 ${M_PI}"/>
+  </xacro:property>
 </robot>

File: mobrob_robin_description/urdf/mobrob_robin_base/base.urdf.xacro (robot description, xacro)
@@ -100,4 +100,9 @@
   <!--                         Wheel definition rotation z-axis                                        -->
   <!--wheel right front rotation z-axis-->
+  <joint name="wheel_rf_rot_z_joint" type="fixed">
+    <origin xyz="${wheel_rf_offset_x} ${wheel_rf_offset_y}  ${base_height}" rpy="0 0 0"/>
+    <parent link="base_link"/>
+    <child link="wheel_rf_rot_z"/>
+  </joint>
   <link name="wheel_rf_rot_z">
     <inertial>
@@ -123,10 +128,10 @@
     </collision>
   </link>
-    <joint name="wheel_rf_rot_z_joint" type="fixed">
-    <origin xyz="${wheel_rf_offset_x} ${wheel_rf_offset_y}  ${base_height}" rpy="0 0 0"/>
-    <parent link="base_link"/>
-    <child link="wheel_rf_rot_z"/>
-  </joint>
     <!--wheel left back rotation z-axis-->
+  <joint name="wheel_lb_rot_z_joint" type="fixed">
+    <origin xyz="${wheel_lb_offset_x} ${wheel_lb_offset_y} ${base_height}" rpy="0 0 0"/>
+    <parent link="base_link"/>
+    <child link="wheel_lb_rot_z"/>
+  </joint>
   <link name="wheel_lb_rot_z">
     <inertial>
@@ -152,10 +157,12 @@
     </collision>
   </link>
-   <joint name="wheel_lb_rot_z_joint" type="fixed">
-    <origin xyz="${wheel_lb_offset_x} ${wheel_lb_offset_y} ${base_height}" rpy="0 0 0"/>
-    <parent link="base_link"/>
-    <child link="wheel_lb_rot_z"/>
-  </joint>
   <!--wheel left front rotation z-axis-->
+  <joint name="wheel_lf_rot_z_joint" type="continuous">
+	<dynamics damping="1.0" friction="0.0" />
+    <origin xyz="${wheel_lf_offset_x} ${wheel_lf_offset_y} ${base_height}" rpy="0 0 0"/>
+    <parent link="base_link"/>
+    <child link="wheel_lf_rot_z"/>
+    <axis xyz="0 0 1"/>
+  </joint>
   <link name="wheel_lf_rot_z">
     <inertial>
@@ -181,12 +188,12 @@
     </collision>
   </link>
-  <joint name="wheel_lf_rot_z_joint" type="continuous">
-  <dynamics damping="1.0" friction="0.0" />
-    <origin xyz="${wheel_lf_offset_x} ${wheel_lf_offset_y} ${base_height}" rpy="0 0 0"/>
-    <parent link="base_link"/>
-    <child link="wheel_lf_rot_z"/>
+  <!--wheel right back rotation z-axis-->
+  <joint name="wheel_rb_rot_z_joint" type="continuous">
+	<dynamics damping="1.0" friction="0.0" />
+    <origin xyz="${wheel_rb_offset_x} ${wheel_rb_offset_y} ${base_height}" rpy="0 0 0"/>
+    <parent link="base_link"/>
+    <child link="wheel_rb_rot_z"/>
     <axis xyz="0 0 1"/>
   </joint>
-  <!--wheel right back rotation z-axis-->
   <link name="wheel_rb_rot_z">
     <inertial>
@@ -212,13 +219,11 @@
     </collision>
   </link>
-  <joint name="wheel_rb_rot_z_joint" type="continuous">
-  <dynamics damping="1.0" friction="0.0" />
-    <origin xyz="${wheel_rb_offset_x} ${wheel_rb_offset_y} ${base_height}" rpy="0 0 0"/>
-    <parent link="base_link"/>
-    <child link="wheel_rb_rot_z"/>
-    <axis xyz="0 0 1"/>
-  </joint>
     <!--                         Wheel definition rotation y-axis                                        -->
     <!--wheel right front rotation y-axis-->
+	<joint name="wheel_rf_rot_y_joint" type="fixed">
+     <origin xyz="0 0 ${wheel_rf_offset_z}" rpy="0 0 0"/>
+     <parent link="wheel_rf_rot_z"/>
+     <child link="wheel_rf_rot_y"/>
+	</joint>
     <link name="wheel_rf_rot_y">
     <inertial>
@@ -242,10 +247,10 @@
     </collision>
   </link>
-   <joint name="wheel_rf_rot_y_joint" type="fixed">
-    <origin xyz="0 0 ${wheel_rf_offset_z}" rpy="0 0 0"/>
-    <parent link="wheel_rf_rot_z"/>
-    <child link="wheel_rf_rot_y"/>
-  </joint>
      <!--wheel left back rotation y-axis-->
+    <joint name="wheel_lb_rot_y_joint" type="fixed">
+		<origin xyz="0 0 ${wheel_lb_offset_z}" rpy="0 0 0"/>
+		<parent link="wheel_lb_rot_z"/>
+		<child link="wheel_lb_rot_y"/>
+	</joint>
     <link name="wheel_lb_rot_y">
     <inertial>
@@ -269,10 +274,10 @@
     </collision>
   </link>
-   <joint name="wheel_lb_rot_y_joint" type="fixed">
-    <origin xyz="0 0 ${wheel_lb_offset_z}" rpy="0 0 0"/>
-    <parent link="wheel_lb_rot_z"/>
-    <child link="wheel_lb_rot_y"/>
-  </joint>
        <!--wheel left front rotation y-axis-->
+    <joint name="wheel_lf_rot_y_joint" type="fixed">
+		<origin xyz="0 0 ${wheel_lf_offset_z}" rpy="0 0 0"/>
+		<parent link="wheel_lf_rot_z"/>
+		<child link="wheel_lf_rot_y"/>
+	</joint>
   <link name="wheel_lf_rot_y">
     <inertial>
@@ -296,10 +301,10 @@
     </collision>
   </link>
-   <joint name="wheel_lf_rot_y_joint" type="fixed">
-    <origin xyz="0 0 ${wheel_lf_offset_z}" rpy="0 0 0"/>
-    <parent link="wheel_lf_rot_z"/>
-    <child link="wheel_lf_rot_y"/>
-  </joint>
          <!--wheel right back rotation y-axis-->
+    <joint name="wheel_rb_rot_y_joint" type="fixed">
+		<origin xyz="0 0 ${wheel_rb_offset_z}" rpy="0 0 0"/>
+		<parent link="wheel_rb_rot_z"/>
+		<child link="wheel_rb_rot_y"/>
+	</joint>
   <link name="wheel_rb_rot_y">
     <inertial>
@@ -323,10 +328,4 @@
     </collision>
   </link>
-   <joint name="wheel_rb_rot_y_joint" type="fixed">
-   <dynamics damping="1.0" friction="0.0" />
-    <origin xyz="0 0 ${wheel_rb_offset_z}" rpy="0 0 0"/>
-    <parent link="wheel_rb_rot_z"/>
-    <child link="wheel_rb_rot_y"/>
-  </joint>
   <xacro:if value="${simulated}">
 	<xacro:mobrob_transmission />
