Commit message: Small update to the urdf modell of the mobrob robot

File: mobrob_robin_description/robots/mobrob.urdf.xacro (robot description, xacro)
@@ -14,7 +14,9 @@
     <insert_block name="ultrasound_sensor2" />
   </xacro:ultrasound_sensor>
+  <!-- not in use
   <xacro:ultrasound_sensor parent="base_link" number="3">
     <insert_block name="ultrasound_sensor3" />
   </xacro:ultrasound_sensor>
+  -->
   <xacro:ultrasound_sensor parent="base_link" number="4">
     <insert_block name="ultrasound_sensor4" />

File: mobrob_robin_description/urdf/mobrob_robin.properties.xacro (robot description, xacro)
@@ -120,9 +120,14 @@
     <origin xyz="${ultrasound_front_side_x} ${ultrasound_left_right_y} ${ultrasound_z}" rpy="0 0 ${M_PI/2}"/>
   </xacro:property>
-  <xacro:property name="ultrasound_sensor3"> <!-- lf front -->
+  <!--
+  <xacro:property name="ultrasound_sensor3">  lf front
     <origin xyz="${ultrasound_front_x} ${ultrasound_back_front_y} ${ultrasound_z}" rpy="0 0 ${0}"/>
   </xacro:property>
-  <xacro:property name="ultrasound_sensor4"> <!-- rf front -->
+  <xacro:property name="ultrasound_sensor4">  rf front
     <origin xyz="${ultrasound_front_x} ${-ultrasound_back_front_y} ${ultrasound_z}" rpy="0 0 ${0}"/>
+  </xacro:property>
+  -->
+  <xacro:property name="ultrasound_sensor4"> <!-- middle front -->
+    <origin xyz="${ultrasound_front_x} 0.0 ${ultrasound_z}" rpy="0 0 ${0}"/>
   </xacro:property>
   <xacro:property name="ultrasound_sensor5"> <!-- rf right -->

Commit message: mobrob_robin_description documentation added

File: mobrob_robin_description/robots/mobrob.urdf.xacro (robot description, xacro)
@@ -1,8 +1,12 @@
 <?xml version="1.0"?>
+<!-- this file builds the mobrob urdf via xacro macros -->
+<!-- it is used for the real and simulated robot urdf model -->
 <robot name="mobrob_robin" xmlns:xacro="http://ros.org/wiki/xacro">
   <xacro:include filename="$(find mobrob_robin_description)/urdf/mobrob_robin.library.xacro" />
   <!-- load the base of the robot   -->
   <xacro:base />
+  <!-- load the sick pls 200 -->
   <xacro:sensor_pls200 />
+  <!-- load the ultrasound sensors -->
   <xacro:ultrasound_sensor parent="base_link" number="0">
     <insert_block name="ultrasound_sensor0" />
@@ -14,5 +18,5 @@
     <insert_block name="ultrasound_sensor2" />
   </xacro:ultrasound_sensor>
-  <!-- not in use
+  <!-- not in use anymore
   <xacro:ultrasound_sensor parent="base_link" number="3">
     <insert_block name="ultrasound_sensor3" />

File: mobrob_robin_description/robots/mobrob_robin_real.urdf.xacro (robot description, xacro)
@@ -1,8 +1,11 @@
 <?xml version="1.0"?>
+<!-- this xacro loads the mobrob robot urdf withouth the gazebo addons -->
 <robot name="mobrob_robin" xmlns:xacro="http://ros.org/wiki/xacro">
+  <!-- this property deactivates the simulation related macros -->
   <xacro:property name="simulated" value="0" />
   <xacro:property name="ofx" value="0" />
-  <xacro:property name="ofx" value="0" />
-  <xacro:property name="ofx" value="0" />
+  <xacro:property name="ofy" value="0" />
+  <xacro:property name="ofz" value="0" />
+  <!-- load the mobrob urdf xacro -->
   <xacro:include filename="$(find mobrob_robin_description)/robots/mobrob.urdf.xacro" />
 </robot>

File: mobrob_robin_description/robots/mobrob_robin_simulated.urdf.xacro (robot description, xacro)
@@ -1,3 +1,4 @@
 <?xml version="1.0"?>
+<!-- THE SIMULATION IS DEPRECATED -->
 <robot name="mobrob_robin" xmlns:xacro="http://ros.org/wiki/xacro">
   <xacro:property name="simulated" value="1" />

File: mobrob_robin_description/urdf/mobrob_robin.common.xacro (robot description, xacro)
@@ -1,3 +1,4 @@
 <?xml version="1.0"?>
+<!-- This files defines some common properties -->
 <robot xmlns:xacro="http://www.ros.org/wiki/xacro">
 	<property name="M_PI" value="3.1415926535897931" />

File: mobrob_robin_description/urdf/mobrob_robin.gazebo.xacro (robot description, xacro)
@@ -1,3 +1,5 @@
 <?xml version="1.0"?>
+<!-- THE SIMULATION IS DEPRECATED -->
+<!-- this file load the gazebo ros controllers -->
 <robot xmlns:xacro="http://www.ros.org/wiki/xacro">
   <gazebo>

File: mobrob_robin_description/urdf/mobrob_robin.library.xacro (robot description, xacro)
@@ -1,13 +1,7 @@
 <?xml version="1.0"?>
-<!--
-  The complete mobrob library of xacros for easy reference
- -->
+<!--  The complete mobrob library of xacros for easy reference-->
 <robot xmlns:xacro="http://ros.org/wiki/xacro">
   <!-- General -->
   <xacro:include filename="$(find mobrob_robin_description)/urdf/mobrob_robin.common.xacro"/>
-  <!-- load gazebo plugins only for simulation -->
-  <xacro:if value="${simulated}">
-    <xacro:include filename="$(find mobrob_robin_description)/urdf/mobrob_robin.gazebo.xacro"/>
-  </xacro:if>
   <!-- Propertiers -->
   <xacro:include filename="$(find mobrob_robin_description)/urdf/mobrob_robin.properties.xacro"/>
@@ -18,3 +12,7 @@
   <!-- Ultrasound -->
   <xacro:include filename="$(find mobrob_robin_description)/urdf/sensors/ultrasound.urdf.xacro"/>
+  <!-- load gazebo plugins only for simulation -->
+  <xacro:if value="${simulated}">
+    <xacro:include filename="$(find mobrob_robin_description)/urdf/mobrob_robin.gazebo.xacro"/>
+  </xacro:if>
 </robot>

File: mobrob_robin_description/urdf/mobrob_robin.properties.xacro (robot description, xacro)
@@ -1,3 +1,4 @@
 <?xml version="1.0"?>
+<!-- This file defines all the used parameters for the urdf model -->
 <robot xmlns:xacro="http://ros.org/wiki/xacro">
   <!--                               Base Parameter                                      -->

File: mobrob_robin_description/urdf/mobrob_robin_base/base.transmission.xacro (robot description, xacro)
@@ -1,3 +1,5 @@
 <?xml version="1.0"?>
+<!-- THE SIMULATION IS DEPRECATED -->
+<!-- this files defines simulation related transmission parameters -->
 <robot xmlns:xacro="http://www.ros.org/wiki/xacro">
   <xacro:macro name="mobrob_transmission">

File: mobrob_robin_description/urdf/mobrob_robin_base/base.urdf.xacro (robot description, xacro)
@@ -1,3 +1,8 @@
 <?xml version="1.0" encoding="UTF-8"?>
+<!-- This maco defines the robots base body -->
+<!-- Starting from the odom frame a x y prismatic joint is added for the xy movement -->
+<!-- A yaw rotary joint follows for rotations around the z axis -->
+<!-- After that the base_link and base_upper joint define the two boxes for the body -->
+<!-- The rest of the file describes the wheel of the robot -->
 <robot xmlns:xacro="http://ros.org/wiki/xacro">
    <xacro:include filename="$(find mobrob_robin_description)/urdf/mobrob_robin_base/base.transmission.xacro" />

File: mobrob_robin_description/urdf/sensors/pls200.gazebo.xacro (robot description, xacro)
@@ -1,3 +1,5 @@
 <?xml version="1.0"?>
+<!-- THE SIMULATION IS DEPRECATED -->
+<!-- This files defines the Sick PLS200 laserscanner for gazebo -->
 <robot xmlns:xacro="http://ros.org/wiki/xacro">
   <gazebo reference="PLS200">

File: mobrob_robin_description/urdf/sensors/pls200.urdf.xacro (robot description, xacro)
@@ -1,3 +1,4 @@
 <?xml version="1.0"?>
+<!-- This file defines the Sick PLS200 visuals -->
 <robot xmlns:xacro="http://ros.org/wiki/xacro">
 	<xacro:if value="${simulated}">

File: mobrob_robin_description/urdf/sensors/ultrasound.urdf.xacro (robot description, xacro)
@@ -1,3 +1,4 @@
 <?xml version="1.0"?>
+<!-- This file defines the ultrasound sensors form and color -->
 <robot xmlns:xacro="http://ros.org/wiki/xacro">
 	<xacro:macro name="ultrasound_sensor" params="number parent *origin">
