Commit message: Added controllers and inverse kinematics to show the movement of the drive wheels in the simulation

File: mobrob_robin_description/urdf/mobrob_robin_base/base.transmission.xacro (robot description, xacro)
@@ -33,24 +33,4 @@
     </transmission>
     <!-- Wheel controllers -->
-    <transmission name="tran_wheel_rf_rot_z">
-        <type>transmission_interface/SimpleTransmission</type>
-        <joint name="wheel_rf_rot_z_joint">
-          <hardwareInterface>PositionJointInterface</hardwareInterface>
-        </joint>
-        <actuator name="motor_wheel_rf_rot_z">
-		  <mechanicalReduction>1</mechanicalReduction>
-          <hardwareInterface>PositionJointInterface</hardwareInterface>
-        </actuator>
-    </transmission>
-    <transmission name="tran_wheel_lb_rot_z">
-        <type>transmission_interface/SimpleTransmission</type>
-        <joint name="wheel_lb_rot_z_joint">
-          <hardwareInterface>PositionJointInterface</hardwareInterface>
-        </joint>
-        <actuator name="motor_wheel_lb_rot_z">
-		  <mechanicalReduction>1</mechanicalReduction>
-          <hardwareInterface>PositionJointInterface</hardwareInterface>
-        </actuator>
-    </transmission>
     <transmission name="tran_wheel_lf_rot_z">
         <type>transmission_interface/SimpleTransmission</type>
@@ -73,44 +53,4 @@
         </actuator>
     </transmission>
-    <transmission name="tran_wheel_rf_rot_y">
-        <type>transmission_interface/SimpleTransmission</type>
-        <joint name="wheel_rf_rot_y_joint">
-          <hardwareInterface>PositionJointInterface</hardwareInterface>
-        </joint>
-        <actuator name="motor_wheel_rf_rot_y">
-		  <mechanicalReduction>1</mechanicalReduction>
-          <hardwareInterface>PositionJointInterface</hardwareInterface>
-        </actuator>
-    </transmission>
-    <transmission name="tran_wheel_lb_rot_y">
-        <type>transmission_interface/SimpleTransmission</type>
-        <joint name="wheel_lb_rot_y_joint">
-          <hardwareInterface>PositionJointInterface</hardwareInterface>
-        </joint>
-        <actuator name="motor_wheel_lb_rot_y_joint">
-		  <mechanicalReduction>1</mechanicalReduction>
-          <hardwareInterface>PositionJointInterface</hardwareInterface>
-        </actuator>
-    </transmission>
-    <transmission name="tran_wheel_lf_rot_y">
-        <type>transmission_interface/SimpleTransmission</type>
-        <joint name="wheel_lf_rot_y_joint">
-          <hardwareInterface>PositionJointInterface</hardwareInterface>
-        </joint>
-        <actuator name="motor_wheel_lf_rot_y">
-		  <mechanicalReduction>1</mechanicalReduction>
-          <hardwareInterface>PositionJointInterface</hardwareInterface>
-        </actuator>
-    </transmission>
-    <transmission name="tran_wheel_rb_rot_y">
-        <type>transmission_interface/SimpleTransmission</type>
-        <joint name="wheel_rb_rot_y_joint">
-          <hardwareInterface>PositionJointInterface</hardwareInterface>
-        </joint>
-        <actuator name="motor_wheel_rb_rot_y">
-		  <mechanicalReduction>1</mechanicalReduction>
-          <hardwareInterface>PositionJointInterface</hardwareInterface>
-        </actuator>
-    </transmission>
 </xacro:macro>
 </robot>

File: mobrob_robin_description/urdf/mobrob_robin_base/base.urdf.xacro (robot description, xacro)
@@ -125,10 +125,8 @@
     </collision>
   </link>
-    <joint name="wheel_rf_rot_z_joint" type="continuous">
-    <dynamics damping="1.0" friction="0.0" />
+    <joint name="wheel_rf_rot_z_joint" type="fixed">
     <origin xyz="${wheel_rf_offset_x} ${wheel_rf_offset_y}  ${base_height}" rpy="0 0 0"/>
     <parent link="base_link"/>
     <child link="wheel_rf_rot_z"/>
-    <axis xyz="0 0 1"/>
   </joint>
     <!--wheel left back rotation z-axis-->
@@ -156,10 +154,8 @@
     </collision>
   </link>
-   <joint name="wheel_lb_rot_z_joint" type="continuous">
-   <dynamics damping="1.0" friction="0.0" />
+   <joint name="wheel_lb_rot_z_joint" type="fixed">
     <origin xyz="${wheel_lb_offset_x} ${wheel_lb_offset_y} ${base_height}" rpy="0 0 0"/>
     <parent link="base_link"/>
     <child link="wheel_lb_rot_z"/>
-    <axis xyz="0 0 1"/>
   </joint>
   <!--wheel left front rotation z-axis-->
@@ -248,10 +244,8 @@
     </collision>
   </link>
-   <joint name="wheel_rf_rot_y_joint" type="continuous">
-   <dynamics damping="1.0" friction="0.0" />
+   <joint name="wheel_rf_rot_y_joint" type="fixed">
     <origin xyz="0 0 ${wheel_rf_offset_z}" rpy="0 0 0"/>
     <parent link="wheel_rf_rot_z"/>
     <child link="wheel_rf_rot_y"/>
-    <axis xyz="0 1 0"/>
   </joint>
      <!--wheel left back rotation y-axis-->
@@ -277,10 +271,8 @@
     </collision>
   </link>
-   <joint name="wheel_lb_rot_y_joint" type="continuous">
-   <dynamics damping="1.0" friction="0.0" />
+   <joint name="wheel_lb_rot_y_joint" type="fixed">
     <origin xyz="0 0 ${wheel_lb_offset_z}" rpy="0 0 0"/>
     <parent link="wheel_lb_rot_z"/>
     <child link="wheel_lb_rot_y"/>
-    <axis xyz="0 1 0"/>
   </joint>
        <!--wheel left front rotation y-axis-->
@@ -306,10 +298,8 @@
     </collision>
   </link>
-   <joint name="wheel_lf_rot_y_joint" type="continuous">
-   <dynamics damping="1.0" friction="0.0" />
+   <joint name="wheel_lf_rot_y_joint" type="fixed">
     <origin xyz="0 0 ${wheel_lf_offset_z}" rpy="0 0 0"/>
     <parent link="wheel_lf_rot_z"/>
     <child link="wheel_lf_rot_y"/>
-    <axis xyz="0 1 0"/>
   </joint>
          <!--wheel right back rotation y-axis-->
@@ -335,10 +325,9 @@
     </collision>
   </link>
-   <joint name="wheel_rb_rot_y_joint" type="continuous">
+   <joint name="wheel_rb_rot_y_joint" type="fixed">
    <dynamics damping="1.0" friction="0.0" />
     <origin xyz="0 0 ${wheel_rb_offset_z}" rpy="0 0 0"/>
     <parent link="wheel_rb_rot_z"/>
     <child link="wheel_rb_rot_y"/>
-    <axis xyz="0 1 0"/>
   </joint>
   <xacro:if value="${simulated}">
